Commit message: 更新块的碰撞几何体尺寸，调整为0.045 x 0.045 x 0.06 添加gazebo的抓取和放置脚本

File: src/robot_arm/urdf/block.urdf.xacro (robot description, xacro)
@@ -12,5 +12,5 @@
     <collision>
       <geometry>
-        <box size="0.04 0.04 0.05"/>
+        <box size="0.045 0.045 0.06"/>
       </geometry>
     </collision>
